File: controll_pannel.sch (KiCad schematic (older format))
At the start: 7 parts, among them P5 CONN_6, SW2 SWITCH_INV, SW3 SWITCH_INV

Commit message: populating boards
Parts:
- SW2: value SWITCH_INV -> ~START~/STOP
- SW3: value SWITCH_INV -> ~FWD~/REV
Changed lines of the file:
@@
 $Descr A4 11693 8268
 encoding utf-8
-Sheet 4 5
+Sheet 3 5
 Title ""
 Date ""
@@
 $EndComp
 $Comp
-L +5V #PWR31
+L +5V #PWR34
 U 1 1 5389AC32
 P 6750 2850
-F 0 "#PWR31" H 6750 2940 20  0001 C CNN
+F 0 "#PWR34" H 6750 2940 20  0001 C CNN
 F 1 "+5V" H 6750 2940 30  0000 C CNN
 F 2 "" H 6750 2850 60  0000 C CNN
@@
 	6750 3350 6750 3450
 $Comp
-L GND #PWR32
+L GND #PWR35
 U 1 1 5389ACDA
 P 6750 3450
-F 0 "#PWR32" H 6750 3450 30  0001 C CNN
+F 0 "#PWR35" H 6750 3450 30  0001 C CNN
 F 1 "GND" H 6750 3380 30  0001 C CNN
 F 2 "" H 6750 3450 60  0000 C CNN
@@
 $EndComp
 $Comp
-L GND #PWR30
+L GND #PWR33
 U 1 1 5389AE05
 P 5950 5250
-F 0 "#PWR30" H 5950 5250 30  0001 C CNN
+F 0 "#PWR33" H 5950 5250 30  0001 C CNN
 F 1 "GND" H 5950 5180 30  0001 C CNN
 F 2 "" H 5950 5250 60  0000 C CNN
@@
 P 5950 4250
 F 0 "SW2" H 5750 4400 50  0000 C CNN
-F 1 "SWITCH_INV" H 5800 4100 50  0000 C CNN
+F 1 "~START~/STOP" H 5800 4100 50  0000 C CNN
 F 2 "" H 5950 4250 60  0000 C CNN
 F 3 "" H 5950 4250 60  0000 C CNN
@@
 P 6350 4250
 F 0 "SW3" H 6150 4400 50  0000 C CNN
-F 1 "SWITCH_INV" H 6200 4100 50  0000 C CNN
+F 1 "~FWD~/REV" H 6200 4100 50  0000 C CNN
 F 2 "" H 6350 4250 60  0000 C CNN
 F 3 "" H 6350 4250 60  0000 C CNN
@@
 	4850 2850 6750 2850
 $Comp
-L +5V #PWR29
+L +5V #PWR32
 U 1 1 5389B0A8
 P 5550 4350
-F 0 "#PWR29" H 5550 4440 20  0001 C CNN
+F 0 "#PWR32" H 5550 4440 20  0001 C CNN
 F 1 "+5V" H 5550 4440 30  0000 C CNN
 F 2 "" H 5550 4350 60  0000 C CNN
@@
 $EndComp
 $Comp
-L +5V #PWR28
+L +5V #PWR31
 U 1 1 5389B0D6
 P 5200 4350
-F 0 "#PWR28" H 5200 4440 20  0001 C CNN
+F 0 "#PWR31" H 5200 4440 20  0001 C CNN
 F 1 "+5V" H 5200 4440 30  0000 C CNN
 F 2 "" H 5200 4350 60  0000 C CNN
