File: dcbus.sch (KiCad schematic (older format))
At the start: 13 parts

Commit message: change polar cap symbol to the more acceptable one
Parts:
- removed C?: CAPAPOL, symbol CAPAPOL
- added C?: CP1, symbol CP1
Changed lines of the file:
@@
 Wire Wire Line
 	5950 4600 8450 4600
-$Comp
-L CAPAPOL C?
-U 1 1 5377D223
-P 8250 4050
-F 0 "C?" H 8300 4150 40  0000 L CNN
-F 1 "CAPAPOL" H 8300 3950 40  0000 L CNN
-F 2 "" H 8350 3900 30  0000 C CNN
-F 3 "" H 8250 4050 300 0000 C CNN
-	1    8250 4050
-	1    0    0    -1
-$EndComp
 Wire Wire Line
 	8250 4250 8250 4700
@@
 	4050 3600 4050 3750
 Connection ~ 4050 3750
+$Comp
+L CP1 C?
+U 1 1 537B9635
+P 8250 4050
+F 0 "C?" H 8300 4150 50  0000 L CNN
+F 1 "CP1" H 8300 3950 50  0000 L CNN
+F 2 "" H 8250 4050 60  0000 C CNN
+F 3 "" H 8250 4050 60  0000 C CNN
+	1    8250 4050
+	1    0    0    -1
+$EndComp
 $EndSCHEMATC

Commit message: add a symbol for common mode choke
Parts:
- removed L? (x2): INDUCTOR_SMALL, symbol INDUCTOR_SMALL
- added T?: COMMON MODE CHOKE, symbol TRANSFO
Other:
- moved on the sheet: C?, D?
Changed lines of the file:
@@
 L BRIDGE D?
 U 1 1 5377D1D0
-P 6800 3550
-F 0 "D?" H 6800 3600 70  0000 C CNN
-F 1 "BRIDGE" H 6800 3500 70  0000 C CNN
-F 2 "" H 6800 3550 60  0000 C CNN
-F 3 "" H 6800 3550 60  0000 C CNN
-	1    6800 3550
-	1    0    0    -1
-$EndComp
-Wire Wire Line
-	5950 3550 5950 4600
-Wire Wire Line
-	5950 4600 8450 4600
-Wire Wire Line
-	8250 4250 8250 4700
+P 8750 3550
+F 0 "D?" H 8750 3600 70  0000 C CNN
+F 1 "BRIDGE" H 8750 3500 70  0000 C CNN
+F 2 "" H 8750 3550 60  0000 C CNN
+F 3 "" H 8750 3550 60  0000 C CNN
+	1    8750 3550
+	1    0    0    -1
+$EndComp
+Wire Wire Line
+	7900 3550 7900 4600
+Wire Wire Line
+	7900 4600 10400 4600
+Wire Wire Line
+	10200 4250 10200 4700
 $Comp
 L CONN_3 K?
@@
 L C C?
 U 1 1 5377D2DA
-P 5100 3150
-F 0 "C?" H 5100 3250 40  0000 L CNN
-F 1 "C" H 5106 3065 40  0000 L CNN
-F 2 "" H 5138 3000 30  0000 C CNN
-F 3 "" H 5100 3150 60  0000 C CNN
-	1    5100 3150
+P 7050 3150
+F 0 "C?" H 7050 3250 40  0000 L CNN
+F 1 "C" H 7056 3065 40  0000 L CNN
+F 2 "" H 7088 3000 30  0000 C CNN
+F 3 "" H 7050 3150 60  0000 C CNN
+	1    7050 3150
 	1    0    0    -1
 $EndComp
@@
 L C C?
 U 1 1 5377D30A
-P 5100 3550
-F 0 "C?" H 5100 3650 40  0000 L CNN
-F 1 "C" H 5106 3465 40  0000 L CNN
-F 2 "" H 5138 3400 30  0000 C CNN
-F 3 "" H 5100 3550 60  0000 C CNN
-	1    5100 3550
-	1    0    0    -1
-$EndComp
-$Comp
-L INDUCTOR_SMALL L?
-U 1 1 5377D36E
-P 4600 2950
-F 0 "L?" H 4600 3050 50  0000 C CNN
-F 1 "INDUCTOR_SMALL" H 4600 2900 50  0000 C CNN
-F 2 "" H 4600 2950 60  0000 C CNN
-F 3 "" H 4600 2950 60  0000 C CNN
-	1    4600 2950
-	1    0    0    -1
-$EndComp
-$Comp
-L INDUCTOR_SMALL L?
-U 1 1 5377D399
-P 4600 3750
-F 0 "L?" H 4600 3850 50  0000 C CNN
-F 1 "INDUCTOR_SMALL" H 4600 3700 50  0000 C CNN
-F 2 "" H 4600 3750 60  0000 C CNN
-F 3 "" H 4600 3750 60  0000 C CNN
-	1    4600 3750
+P 7050 3550
+F 0 "C?" H 7050 3650 40  0000 L CNN
+F 1 "C" H 7056 3465 40  0000 L CNN
+F 2 "" H 7088 3400 30  0000 C CNN
+F 3 "" H 7050 3550 60  0000 C CNN
+	1    7050 3550
 	1    0    0    -1
 $EndComp
@@
 	4350 3750 4350 3550
 Wire Wire Line
-	4850 2950 5100 2950
-Wire Wire Line
-	4850 3750 5100 3750
-Wire Wire Line
-	3600 2950 4350 2950
-Wire Wire Line
-	3600 3750 4350 3750
+	5150 2950 7050 2950
+Wire Wire Line
+	5150 3750 7050 3750
+Wire Wire Line
+	3600 2950 4750 2950
+Wire Wire Line
+	3600 3750 4750 3750
 Wire Wire Line
 	3700 3600 3700 3750
@@
 L GNDPWR #PWR?
 U 1 1 5377D78A
-P 5300 3400
-F 0 "#PWR?" H 5300 3450 40  0001 C CNN
-F 1 "GNDPWR" H 5300 3320 40  0000 C CNN
-F 2 "" H 5300 3400 60  0000 C CNN
-F 3 "" H 5300 3400 60  0000 C CNN
-	1    5300 3400
-	1    0    0    -1
-$EndComp
-Wire Wire Line
-	5100 3350 5300 3350
-Wire Wire Line
-	5300 3350 5300 3400
-Wire Wire Line
-	5100 2950 5100 2700
-Wire Wire Line
-	5100 2700 6800 2700
-Wire Wire Line
-	5100 3750 5100 4400
-Wire Wire Line
-	5100 4400 6800 4400
+P 7250 3400
+F 0 "#PWR?" H 7250 3450 40  0001 C CNN
+F 1 "GNDPWR" H 7250 3320 40  0000 C CNN
+F 2 "" H 7250 3400 60  0000 C CNN
+F 3 "" H 7250 3400 60  0000 C CNN
+	1    7250 3400
+	1    0    0    -1
+$EndComp
+Wire Wire Line
+	7050 3350 7250 3350
+Wire Wire Line
+	7250 3350 7250 3400
+Wire Wire Line
+	7050 2950 7050 2700
+Wire Wire Line
+	7050 2700 8750 2700
+Wire Wire Line
+	7050 3750 7050 4400
+Wire Wire Line
+	7050 4400 8750 4400
 $Comp
 L GND #PWR?
 U 1 1 5377D7C9
-P 8250 4700
-F 0 "#PWR?" H 8250 4700 30  0001 C CNN
-F 1 "GND" H 8250 4630 30  0001 C CNN
-F 2 "" H 8250 4700 60  0000 C CNN
-F 3 "" H 8250 4700 60  0000 C CNN
-	1    8250 4700
-	1    0    0    -1
-$EndComp
-Connection ~ 8250 4600
+P 10200 4700
+F 0 "#PWR?" H 10200 4700 30  0001 C CNN
+F 1 "GND" H 10200 4630 30  0001 C CNN
+F 2 "" H 10200 4700 60  0000 C CNN
+F 3 "" H 10200 4700 60  0000 C CNN
+	1    10200 4700
+	1    0    0    -1
+$EndComp
+Connection ~ 10200 4600
 Wire Wire Line
 	2100 3200 2100 2950
@@
 Wire Wire Line
 	2250 3750 3100 3750
-Text HLabel 8450 3550 2    60   Input ~ 0
+Text HLabel 10400 3550 2    60   Input ~ 0
 DCBUS
 Wire Wire Line
-	8250 3550 8450 3550
-Text HLabel 8450 4600 2    60   Input ~ 0
+	10200 3550 10400 3550
+Text HLabel 10400 4600 2    60   Input ~ 0
 GND
 Text HLabel 1950 3850 0    60   Input ~ 0
@@
 L INDUCTOR L?
 U 1 1 5377DB56
-P 7950 3550
-F 0 "L?" V 7900 3550 40  0000 C CNN
-F 1 "INDUCTOR" V 8050 3550 40  0000 C CNN
-F 2 "" H 7950 3550 60  0000 C CNN
-F 3 "" H 7950 3550 60  0000 C CNN
-	1    7950 3550
+P 9900 3550
+F 0 "L?" V 9850 3550 40  0000 C CNN
+F 1 "INDUCTOR" V 10000 3550 40  0000 C CNN
+F 2 "" H 9900 3550 60  0000 C CNN
+F 3 "" H 9900 3550 60  0000 C CNN
+	1    9900 3550
 	0    -1   -1   0
 $EndComp
 Wire Wire Line
-	8250 3550 8250 3850
+	10200 3550 10200 3850
 $Comp
 L R R?
@@
 L CP1 C?
 U 1 1 537B9635
-P 8250 4050
-F 0 "C?" H 8300 4150 50  0000 L CNN
-F 1 "CP1" H 8300 3950 50  0000 L CNN
-F 2 "" H 8250 4050 60  0000 C CNN
-F 3 "" H 8250 4050 60  0000 C CNN
-	1    8250 4050
-	1    0    0    -1
-$EndComp
+P 10200 4050
+F 0 "C?" H 10250 4150 50  0000 L CNN
+F 1 "CP1" H 10250 3950 50  0000 L CNN
+F 2 "" H 10200 4050 60  0000 C CNN
+F 3 "" H 10200 4050 60  0000 C CNN
+	1    10200 4050
+	1    0    0    -1
+$EndComp
+$Comp
+L TRANSFO T?
+U 1 1 537B9702
+P 4950 3350
+F 0 "T?" H 4950 3600 70  0000 C CNN
+F 1 "COMMON MODE CHOKE" H 4950 3050 70  0000 C CNN
+F 2 "" H 4950 3350 60  0000 C CNN
+F 3 "" H 4950 3350 60  0000 C CNN
+	1    4950 3350
+	0    -1   -1   0
+$EndComp
+Connection ~ 4350 3750
+Connection ~ 4350 2950
 $EndSCHEMATC

Commit message: add placeholder for controll schematics
Connections:
- wire segments 28 -> 36
Other:
- moved on the sheet: C?, D?, K?
Changed lines of the file:
@@
 $Descr A4 11693 8268
 encoding utf-8
-Sheet 2 2
+Sheet 2 3
 Title ""
 Date ""
@@
 L BRIDGE D?
 U 1 1 5377D1D0
-P 8750 3550
-F 0 "D?" H 8750 3600 70  0000 C CNN
-F 1 "BRIDGE" H 8750 3500 70  0000 C CNN
-F 2 "" H 8750 3550 60  0000 C CNN
-F 3 "" H 8750 3550 60  0000 C CNN
-	1    8750 3550
-	1    0    0    -1
-$EndComp
-Wire Wire Line
-	7900 3550 7900 4600
-Wire Wire Line
-	7900 4600 10400 4600
-Wire Wire Line
-	10200 4250 10200 4700
+P 7300 3550
+F 0 "D?" H 7300 3600 70  0000 C CNN
+F 1 "BRIDGE" H 7300 3500 70  0000 C CNN
+F 2 "" H 7300 3550 60  0000 C CNN
+F 3 "" H 7300 3550 60  0000 C CNN
+	1    7300 3550
+	1    0    0    -1
+$EndComp
+Wire Wire Line
+	6450 3550 6450 4600
+Wire Wire Line
+	6450 4600 8750 4600
+Wire Wire Line
+	8750 4600 8950 4600
+Wire Wire Line
+	8750 4250 8750 4600
+Wire Wire Line
+	8750 4600 8750 4700
 $Comp
 L CONN_3 K?
 U 1 1 5377D28E
-P 1750 3300
-F 0 "K?" V 1700 3300 50  0000 C CNN
-F 1 "CONN_3" V 1800 3300 40  0000 C CNN
-F 2 "" H 1750 3300 60  0000 C CNN
-F 3 "" H 1750 3300 60  0000 C CNN
-	1    1750 3300
+P 2250 3300
+F 0 "K?" V 2200 3300 50  0000 C CNN
+F 1 "CONN_3" V 2300 3300 40  0000 C CNN
+F 2 "" H 2250 3300 60  0000 C CNN
+F 3 "" H 2250 3300 60  0000 C CNN
+	1    2250 3300
 	-1   0    0    1
 $EndComp
@@
 L GNDPWR #PWR?
 U 1 1 5377D2AD
-P 2100 3850
-F 0 "#PWR?" H 2100 3900 40  0001 C CNN
-F 1 "GNDPWR" H 2100 3770 40  0000 C CNN
-F 2 "" H 2100 3850 60  0000 C CNN
-F 3 "" H 2100 3850 60  0000 C CNN
-	1    2100 3850
-	1    0    0    -1
-$EndComp
-Wire Wire Line
-	2100 3400 2100 3850
+P 2600 3850
+F 0 "#PWR?" H 2600 3900 40  0001 C CNN
+F 1 "GNDPWR" H 2600 3770 40  0000 C CNN
+F 2 "" H 2600 3850 60  0000 C CNN
+F 3 "" H 2600 3850 60  0000 C CNN
+	1    2600 3850
+	1    0    0    -1
+$EndComp
+Wire Wire Line
+	2600 3400 2600 3850
 $Comp
 L C C?
@@
 L C C?
 U 1 1 5377D2DA
-P 7050 3150
-F 0 "C?" H 7050 3250 40  0000 L CNN
-F 1 "C" H 7056 3065 40  0000 L CNN
-F 2 "" H 7088 3000 30  0000 C CNN
-F 3 "" H 7050 3150 60  0000 C CNN
-	1    7050 3150
+P 5600 3150
+F 0 "C?" H 5600 3250 40  0000 L CNN
+F 1 "C" H 5606 3065 40  0000 L CNN
+F 2 "" H 5638 3000 30  0000 C CNN
+F 3 "" H 5600 3150 60  0000 C CNN
+	1    5600 3150
 	1    0    0    -1
 $EndComp
@@
 L C C?
 U 1 1 5377D30A
-P 7050 3550
-F 0 "C?" H 7050 3650 40  0000 L CNN
-F 1 "C" H 7056 3465 40  0000 L CNN
-F 2 "" H 7088 3400 30  0000 C CNN
-F 3 "" H 7050 3550 60  0000 C CNN
-	1    7050 3550
+P 5600 3550
+F 0 "C?" H 5600 3650 40  0000 L CNN
+F 1 "C" H 5606 3465 40  0000 L CNN
+F 2 "" H 5638 3400 30  0000 C CNN
+F 3 "" H 5600 3550 60  0000 C CNN
+	1    5600 3550
 	1    0    0    -1
 $EndComp
@@
 	4350 3750 4350 3550
 Wire Wire Line
-	5150 2950 7050 2950
-Wire Wire Line
-	5150 3750 7050 3750
-Wire Wire Line
-	3600 2950 4750 2950
-Wire Wire Line
-	3600 3750 4750 3750
+	5150 2950 5600 2950
+Wire Wire Line
+	5150 3750 5600 3750
+Wire Wire Line
+	3600 2950 3700 2950
+Wire Wire Line
+	3700 2950 4050 2950
+Wire Wire Line
+	4050 2950 4350 2950
+Wire Wire Line
+	4350 2950 4750 2950
+Wire Wire Line
+	3600 3750 3700 3750
+Wire Wire Line
+	3700 3750 4050 3750
+Wire Wire Line
+	4050 3750 4350 3750
+Wire Wire Line
+	4350 3750 4750 3750
 Wire Wire Line
 	3700 3600 3700 3750
@@
 L GNDPWR #PWR?
 U 1 1 5377D78A
-P 7250 3400
-F 0 "#PWR?" H 7250 3450 40  0001 C CNN
-F 1 "GNDPWR" H 7250 3320 40  0000 C CNN
-F 2 "" H 7250 3400 60  0000 C CNN
-F 3 "" H 7250 3400 60  0000 C CNN
-	1    7250 3400
-	1    0    0    -1
-$EndComp
-Wire Wire Line
-	7050 3350 7250 3350
-Wire Wire Line
-	7250 3350 7250 3400
-Wire Wire Line
-	7050 2950 7050 2700
-Wire Wire Line
-	7050 2700 8750 2700
-Wire Wire Line
-	7050 3750 7050 4400
-Wire Wire Line
-	7050 4400 8750 4400
+P 5800 3400
+F 0 "#PWR?" H 5800 3450 40  0001 C CNN
+F 1 "GNDPWR" H 5800 3320 40  0000 C CNN
+F 2 "" H 5800 3400 60  0000 C CNN
+F 3 "" H 5800 3400 60  0000 C CNN
+	1    5800 3400
+	1    0    0    -1
+$EndComp
+Wire Wire Line
+	5600 3350 5800 3350
+Wire Wire Line
+	5800 3350 5800 3400
+Wire Wire Line
+	5600 2950 5600 2700
+Wire Wire Line
+	5600 2700 7300 2700
+Wire Wire Line
+	5600 3750 5600 4400
+Wire Wire Line
+	5600 4400 7300 4400
 $Comp
 L GND #PWR?
 U 1 1 5377D7C9
-P 10200 4700
-F 0 "#PWR?" H 10200 4700 30  0001 C CNN
-F 1 "GND" H 10200 4630 30  0001 C CNN
-F 2 "" H 10200 4700 60  0000 C CNN
-F 3 "" H 10200 4700 60  0000 C CNN
-	1    10200 4700
-	1    0    0    -1
-$EndComp
-Connection ~ 10200 4600
-Wire Wire Line
-	2100 3200 2100 2950
-Wire Wire Line
-	2100 2950 3100 2950
-Wire Wire Line
-	2100 3300 2250 3300
-Wire Wire Line
-	2250 3300 2250 3750
-Wire Wire Line
-	2250 3750 3100 3750
-Text HLabel 10400 3550 2    60   Input ~ 0
+P 8750 4700
+F 0 "#PWR?" H 8750 4700 30  0001 C CNN
+F 1 "GND" H 8750 4630 30  0001 C CNN
+F 2 "" H 8750 4700 60  0000 C CNN
+F 3 "" H 8750 4700 60  0000 C CNN
+	1    8750 4700
+	1    0    0    -1
+$EndComp
+Connection ~ 8750 4600
+Wire Wire Line
+	2600 3200 2600 2950
+Wire Wire Line
+	2600 2950 3100 2950
+Wire Wire Line
+	2600 3300 2750 3300
+Wire Wire Line
+	2750 3300 2750 3750
+Wire Wire Line
+	2750 3750 3100 3750
+Text HLabel 8950 3550 2    60   Input ~ 0
 DCBUS
 Wire Wire Line
-	10200 3550 10400 3550
-Text HLabel 10400 4600 2    60   Input ~ 0
+	8750 3550 8950 3550
+Text HLabel 8950 4600 2    60   Input ~ 0
 GND
-Text HLabel 1950 3850 0    60   Input ~ 0
+Text HLabel 2450 3850 0    60   Input ~ 0
 EARTH
 Wire Wire Line
-	2100 3850 1950 3850
+	2600 3850 2450 3850
 $Comp
 L INDUCTOR L?
 U 1 1 5377DB56
-P 9900 3550
-F 0 "L?" V 9850 3550 40  0000 C CNN
-F 1 "INDUCTOR" V 10000 3550 40  0000 C CNN
-F 2 "" H 9900 3550 60  0000 C CNN
-F 3 "" H 9900 3550 60  0000 C CNN
-	1    9900 3550
+P 8450 3550
+F 0 "L?" V 8400 3550 40  0000 C CNN
+F 1 "INDUCTOR" V 8550 3550 40  0000 C CNN
+F 2 "" H 8450 3550 60  0000 C CNN
+F 3 "" H 8450 3550 60  0000 C CNN
+	1    8450 3550
 	0    -1   -1   0
 $EndComp
 Wire Wire Line
-	10200 3550 10200 3850
+	8750 3550 8750 3850
 $Comp
 L R R?
@@
 L CP1 C?
 U 1 1 537B9635
-P 10200 4050
-F 0 "C?" H 10250 4150 50  0000 L CNN
-F 1 "CP1" H 10250 3950 50  0000 L CNN
-F 2 "" H 10200 4050 60  0000 C CNN
-F 3 "" H 10200 4050 60  0000 C CNN
-	1    10200 4050
-	1    0    0    -1
-$EndComp
+P 8750 4050
+F 0 "C?" H 8800 4150 50  0000 L CNN
+F 1 "CP1" H 8800 3950 50  0000 L CNN
+F 2 "" H 8750 4050 60  0000 C CNN
+F 3 "" H 8750 4050 60  0000 C CNN
+	1    8750 4050
+	1    0    0    -1
+$EndComp

Commit message: add snubbing, mov for the main cap protection and a bleeder resistor for the main cap. add annotations finally
Parts:
- removed L?: INDUCTOR, symbol INDUCTOR
- added C5: C, symbol C
- added R2, R3: R, symbol R
- added VR2: VR, symbol VR
- gave numbers to parts that had none: 11
Connections:
- wire segments 36 -> 33
Other:
- moved on the sheet: D1
Changed lines of the file:
@@
 $EndDescr
 $Comp
-L BRIDGE D?
+L BRIDGE D1
 U 1 1 5377D1D0
-P 7300 3550
-F 0 "D?" H 7300 3600 70  0000 C CNN
-F 1 "BRIDGE" H 7300 3500 70  0000 C CNN
-F 2 "" H 7300 3550 60  0000 C CNN
-F 3 "" H 7300 3550 60  0000 C CNN
-	1    7300 3550
-	1    0    0    -1
-$EndComp
-Wire Wire Line
-	6450 3550 6450 4600
-Wire Wire Line
-	6450 4600 8750 4600
-Wire Wire Line
-	8750 4600 8950 4600
-Wire Wire Line
-	8750 4250 8750 4600
-Wire Wire Line
-	8750 4600 8750 4700
-$Comp
-L CONN_3 K?
+P 6900 3550
+F 0 "D1" H 6900 3600 70  0000 C CNN
+F 1 "BRIDGE" H 6900 3500 70  0000 C CNN
+F 2 "" H 6900 3550 60  0000 C CNN
+F 3 "" H 6900 3550 60  0000 C CNN
+	1    6900 3550
+	1    0    0    -1
+$EndComp
+Wire Wire Line
+	6050 3550 6050 4600
+Wire Wire Line
+	6050 4600 9600 4600
+Wire Wire Line
+	8750 4250 8750 4700
+$Comp
+L CONN_3 K1
 U 1 1 5377D28E
 P 2250 3300
-F 0 "K?" V 2200 3300 50  0000 C CNN
+F 0 "K1" V 2200 3300 50  0000 C CNN
 F 1 "CONN_3" V 2300 3300 40  0000 C CNN
 F 2 "" H 2250 3300 60  0000 C CNN
@@
 $EndComp
 $Comp
-L GNDPWR #PWR?
+L GNDPWR #PWR1
 U 1 1 5377D2AD
 P 2600 3850
-F 0 "#PWR?" H 2600 3900 40  0001 C CNN
+F 0 "#PWR1" H 2600 3900 40  0001 C CNN
 F 1 "GNDPWR" H 2600 3770 40  0000 C CNN
 F 2 "" H 2600 3850 60  0000 C CNN
@@
 	2600 3400 2600 3850
 $Comp
-L C C?
+L C C1
 U 1 1 5377D2CB
 P 4350 3350
-F 0 "C?" H 4350 3450 40  0000 L CNN
+F 0 "C1" H 4350 3450 40  0000 L CNN
 F 1 "C" H 4356 3265 40  0000 L CNN
 F 2 "" H 4388 3200 30  0000 C CNN
@@
 $EndComp
 $Comp
-L C C?
+L C C2
 U 1 1 5377D2DA
 P 5600 3150
-F 0 "C?" H 5600 3250 40  0000 L CNN
+F 0 "C2" H 5600 3250 40  0000 L CNN
 F 1 "C" H 5606 3065 40  0000 L CNN
 F 2 "" H 5638 3000 30  0000 C CNN
@@
 $EndComp
 $Comp
-L C C?
+L C C3
 U 1 1 5377D30A
 P 5600 3550
-F 0 "C?" H 5600 3650 40  0000 L CNN
+F 0 "C3" H 5600 3650 40  0000 L CNN
 F 1 "C" H 5606 3465 40  0000 L CNN
 F 2 "" H 5638 3400 30  0000 C CNN
@@
 $EndComp
 $Comp
-L VR VR?
+L VR VR1
 U 1 1 5377D409
 P 3700 3350
-F 0 "VR?" V 3760 3304 40  0000 C TNN
+F 0 "VR1" V 3760 3304 40  0000 C TNN
 F 1 "VR" V 3700 3350 40  0000 C CNN
 F 2 "" H 3700 3350 60  0000 C CNN
@@
 $EndComp
 $Comp
-L FUSE F?
+L FUSE F1
 U 1 1 5377D438
 P 3350 2950
-F 0 "F?" H 3450 3000 40  0000 C CNN
+F 0 "F1" H 3450 3000 40  0000 C CNN
 F 1 "FUSE" H 3250 2900 40  0000 C CNN
 F 2 "" H 3350 2950 60  0000 C CNN
@@
 $EndComp
 $Comp
-L THERMISTOR TH?
+L THERMISTOR TH1
 U 1 1 5377D447
 P 3350 3750
-F 0 "TH?" V 3450 3800 50  0000 C CNN
+F 0 "TH1" V 3450 3800 50  0000 C CNN
 F 1 "THERMISTOR" V 3250 3750 50  0000 C CNN
 F 2 "" H 3350 3750 60  0000 C CNN
@@
 	5150 3750 5600 3750
 Wire Wire Line
-	3600 2950 3700 2950
-Wire Wire Line
-	3700 2950 4050 2950
-Wire Wire Line
-	4050 2950 4350 2950
-Wire Wire Line
-	4350 2950 4750 2950
-Wire Wire Line
-	3600 3750 3700 3750
-Wire Wire Line
-	3700 3750 4050 3750
-Wire Wire Line
-	4050 3750 4350 3750
-Wire Wire Line
-	4350 3750 4750 3750
+	3600 2950 4750 2950
+Wire Wire Line
+	3600 3750 4750 3750
 Wire Wire Line
 	3700 3600 3700 3750
@@
 Connection ~ 3700 2950
 $Comp
-L GNDPWR #PWR?
+L GNDPWR #PWR2
 U 1 1 5377D78A
 P 5800 3400
-F 0 "#PWR?" H 5800 3450 40  0001 C CNN
+F 0 "#PWR2" H 5800 3450 40  0001 C CNN
 F 1 "GNDPWR" H 5800 3320 40  0000 C CNN
 F 2 "" H 5800 3400 60  0000 C CNN
@@
 	5600 2950 5600 2700
 Wire Wire Line
-	5600 2700 7300 2700
+	5600 2700 6900 2700
 Wire Wire Line
 	5600 3750 5600 4400
 Wire Wire Line
-	5600 4400 7300 4400
-$Comp
-L GND #PWR?
+	5600 4400 6900 4400
+$Comp
+L GND #PWR3
 U 1 1 5377D7C9
 P 8750 4700
-F 0 "#PWR?" H 8750 4700 30  0001 C CNN
+F 0 "#PWR3" H 8750 4700 30  0001 C CNN
 F 1 "GND" H 8750 4630 30  0001 C CNN
 F 2 "" H 8750 4700 60  0000 C CNN
@@
 Wire Wire Line
 	2750 3750 3100 3750
-Text HLabel 8950 3550 2    60   Input ~ 0
+Text HLabel 9550 3550 2    60   Input ~ 0
 DCBUS
 Wire Wire Line
-	8750 3550 8950 3550
-Text HLabel 8950 4600 2    60   Input ~ 0
+	7750 3550 9550 3550
+Text HLabel 9600 4600 2    60   Input ~ 0
 GND
 Text HLabel 2450 3850 0    60   Input ~ 0
@@
 Wire Wire Line
 	2600 3850 2450 3850
-$Comp
-L INDUCTOR L?
-U 1 1 5377DB56
-P 8450 3550
-F 0 "L?" V 8400 3550 40  0000 C CNN
-F 1 "INDUCTOR" V 8550 3550 40  0000 C CNN
-F 2 "" H 8450 3550 60  0000 C CNN
-F 3 "" H 8450 3550 60  0000 C CNN
-	1    8450 3550
-	0    -1   -1   0
-$EndComp
 Wire Wire Line
 	8750 3550 8750 3850
 $Comp
-L R R?
+L R R1
 U 1 1 5377DD0E
 P 4050 3350
-F 0 "R?" V 4130 3350 40  0000 C CNN
+F 0 "R1" V 4130 3350 40  0000 C CNN
 F 1 "1.5M 1W" V 4057 3351 40  0000 C CNN
 F 2 "" V 3980 3350 30  0000 C CNN
@@
 Connection ~ 4050 3750
 $Comp
-L CP1 C?
+L CP1 C4
 U 1 1 537B9635
 P 8750 4050
-F 0 "C?" H 8800 4150 50  0000 L CNN
+F 0 "C4" H 8800 4150 50  0000 L CNN
 F 1 "CP1" H 8800 3950 50  0000 L CNN
 F 2 "" H 8750 4050 60  0000 C CNN
@@
 $EndComp
 $Comp
-L TRANSFO T?
+L TRANSFO T1
 U 1 1 537B9702
 P 4950 3350
-F 0 "T?" H 4950 3600 70  0000 C CNN
+F 0 "T1" H 4950 3600 70  0000 C CNN
 F 1 "COMMON MODE CHOKE" H 4950 3050 70  0000 C CNN
 F 2 "" H 4950 3350 60  0000 C CNN
@@
 Connection ~ 4350 3750
 Connection ~ 4350 2950
+$Comp
+L VR VR2
+U 1 1 537E750E
+P 9150 4050
+F 0 "VR2" V 9210 4004 40  0000 C TNN
+F 1 "VR" V 9150 4050 40  0000 C CNN
+F 2 "" H 9150 4050 60  0000 C CNN
+F 3 "" H 9150 4050 60  0000 C CNN
+	1    9150 4050
+	1    0    0    -1
+$EndComp
+Wire Wire Line
+	9150 3800 9150 3550
+Connection ~ 9150 3550
+Wire Wire Line
+	9150 4300 9150 4600
+Connection ~ 9150 4600
+$Comp
+L C C5
+U 1 1 537E76B1
+P 9400 4400
+F 0 "C5" H 9400 4500 40  0000 L CNN
+F 1 "C" H 9406 4315 40  0000 L CNN
+F 2 "" H 9438 4250 30  0000 C CNN
+F 3 "" H 9400 4400 60  0000 C CNN
+	1    9400 4400
+	1    0    0    -1
+$EndComp
+$Comp
+L R R3
+U 1 1 537E777F
+P 9400 3950
+F 0 "R3" V 9480 3950 40  0000 C CNN
+F 1 "R" V 9407 3951 40  0000 C CNN
+F 2 "" V 9330 3950 30  0000 C CNN
+F 3 "" H 9400 3950 30  0000 C CNN
+	1    9400 3950
+	1    0    0    -1
+$EndComp
+Wire Wire Line
+	9400 3700 9400 3550
+Connection ~ 9400 3550
+Connection ~ 8750 3550
+$Comp
+L R R2
+U 1 1 537E7ACB
+P 8350 4100
+F 0 "R2" V 8430 4100 40  0000 C CNN
+F 1 "R" V 8357 4101 40  0000 C CNN
+F 2 "" V 8280 4100 30  0000 C CNN
+F 3 "" H 8350 4100 30  0000 C CNN
+	1    8350 4100
+	1    0    0    -1
+$EndComp
+Wire Wire Line
+	8350 3850 8350 3550
+Connection ~ 8350 3550
+Wire Wire Line
+	8350 4350 8350 4600
+Connection ~ 8350 4600
 $EndSCHEMATC
