File: output.sch (KiCad schematic (older format))
At the start: 10 parts

Commit message: populating boards
Parts:
- added C? (x7): 1n, symbol C
- added C? (x5): C, symbol C
- added C?: CP1, symbol CP1
- added R? (x14): 100R, symbol R
- added R? (x6): R, symbol R
- gave numbers to parts that had none: 10
Connections:
- net labels added: DCBUS, FAULT, PWM_U_BOT, PWM_U_TOP, PWM_V_BOT, PWM_V_TOP, PWM_W_BOT, PWM_W_TOP, SHORT_PROTECT, U_CURRENT, V_CURRENT, W_CURRENT
- wire segments 26 -> 74
